File: Ember.kicad_sch (KiCad schematic)
At the start: 0 parts

Commit message: FInished initial schematic
Parts:
- added C1, C2, C3, C4, C5, C6, C7, C8: 1uF, symbol Device:C
- added C10: 10uF, symbol Device:C
- added C9: 100nF, symbol Device:C
- added J1: FT232H Control, Connector_PinHeader_2.54mm:PinHeader_1x11_P2.54mm_Vertical, symbol Connector:Conn_01x11_Pin
- added J2: FT232H Power + Data, Connector_PinHeader_2.54mm:PinHeader_1x11_P2.54mm_Vertical, symbol Connector:Conn_01x11_Pin
- added J3: LCD Panel - 28 Pin Tail, Package_DIP:DIP-20_W7.62mm, symbol Connector_Generic:Conn_01x28
- added J4: Conn_01x02_Pin, Package_DIP:DIP-20_W7.62mm, symbol Connector:Conn_01x02_Pin
- added J5: Spare GPIO, Package_DIP:DIP-20_W7.62mm, symbol Connector:Conn_01x02_Pin
- added J6: LCD backup - wire pads, symbol Connector_Generic:Conn_02x14_Top_Bottom
- added Q1: 2N2222A, symbol Transistor_BJT:Q_NPN_BCE
- added R1: 220, symbol Device:R
- added R2: 1k, symbol Device:R
- added R3: 10k, symbol Device:R
Connections:
- new net: J4.1 (Pin_1), R1.2
- new net: J4.2 (Pin_2), Q1.2 (C)
- new net: Q1.1 (B), R2.2, R3.1
- new net +3V3: C10.1, C9.1, J2.1 (Pin_1), J3.1 (Pin_1), J3.15 (Pin_15), J6.1 (Pin_1), J6.15 (Pin_15)
- new net +5V: J2.2 (Pin_2), R1.1
- new net BIAS3: C1.1, J3.3 (Pin_3), J6.3 (Pin_3)
- new net BIAS4: C2.1, J3.4 (Pin_4), J6.4 (Pin_4)
- new net BIAS5: C3.1, J3.5 (Pin_5), J6.5 (Pin_5)
- new net BIAS6: C4.1, J3.6 (Pin_6), J6.6 (Pin_6)
- new net BIAS7: C5.1, J3.7 (Pin_7), J6.7 (Pin_7)
- new net C0: J1.11 (Pin_22), J3.24 (Pin_24), J6.24 (Pin_24)
- new net C1: J1.10 (Pin_21), J3.25 (Pin_25), J6.25 (Pin_25)
- new net C2: J1.9 (Pin_20), J3.26 (Pin_26), J6.26 (Pin_26)
- new net C3: J1.8 (Pin_19), J3.27 (Pin_27), J6.27 (Pin_27)
- new net C4: J1.7 (Pin_18), J3.28 (Pin_28), J6.28 (Pin_28)
- new net C5: J1.6 (Pin_17), R2.1
- new net C6: J1.5 (Pin_16), J5.1 (Pin_1)
- new net C7: J1.4 (Pin_15), J5.2 (Pin_2)
- new net D0: J2.4 (Pin_4), J3.23 (Pin_23), J6.23 (Pin_23)
- new net D1: J2.5 (Pin_5), J3.22 (Pin_22), J6.22 (Pin_22)
- new net D2: J2.6 (Pin_6), J3.21 (Pin_21), J6.21 (Pin_21)
- new net D3: J2.7 (Pin_7), J3.20 (Pin_20), J6.20 (Pin_20)
- new net D4: J2.8 (Pin_8), J3.19 (Pin_19), J6.19 (Pin_19)
- new net D5: J2.9 (Pin_9), J3.18 (Pin_18), J6.18 (Pin_18)
- new net D6: J2.10 (Pin_10), J3.17 (Pin_17), J6.17 (Pin_17)
- new net D7: J2.11 (Pin_11), J3.16 (Pin_16), J6.16 (Pin_16)
- new net GND: C1.2, C10.2, C2.2, C3.2, C4.2, C5.2, C8.2, C9.2, J1.1 (Pin_12), J2.3 (Pin_3), J3.14 (Pin_14), J3.2 (Pin_2), J6.14 (Pin_14), J6.2 (Pin_2), Q1.3 (E), R3.2
- new net PUMP_10: C7.1, J3.10 (Pin_10), J6.10 (Pin_10)
- new net PUMP_11: C7.2, J3.11 (Pin_11), J6.11 (Pin_11)
- new net PUMP_12_13: C8.1, J3.12 (Pin_12), J3.13 (Pin_13), J6.12 (Pin_12), J6.13 (Pin_13)
- new net PUMP_8: C6.1, J3.8 (Pin_8), J6.8 (Pin_8)
- new net PUMP_9: C6.2, J3.9 (Pin_9), J6.9 (Pin_9)
- no-connect marks 0 -> 2
Other:
- note added: "1 = A (red) 2 = K (black)"
- note added: "24=/RD 25=/WR 26=A0 27=/RES 28=/CS"
- note added: "For ERC - not a circuit"
- title: (none) -> Ember

Commit message: Built the whole v1.0 design in one day
Parts:
- C1, C2, C3, C4, C5, C6, C7, C8, C9: footprint (none) -> Capacitor_THT:C_Disc_D4.7mm_W2.5mm_P5.00mm
- C10: footprint (none) -> Capacitor_THT:CP_Radial_D5.0mm_P2.50mm; symbol Device:C -> Device:C_Polarized
- J1, J2: footprint Connector_PinHeader_2.54mm:PinHeader_1x11_P2.54mm_Vertical -> Connector_PinSocket_2.54mm:PinSocket_1x11_P2.54mm_Vertical
- J3: footprint Package_DIP:DIP-20_W7.62mm -> Connector_FFC-FPC:Hirose_FH12-28S-0.5SH_1x28-1MP_P0.50mm_Horizontal
- J4: value Conn_01x02_Pin -> LCD Backlight; footprint Package_DIP:DIP-20_W7.62mm -> Connector_PinSocket_2.54mm:PinSocket_1x02_P2.54mm_Horizontal
- J5: footprint Package_DIP:DIP-20_W7.62mm -> Connector_PinHeader_2.54mm:PinHeader_1x02_P2.54mm_Vertical
- J6: footprint (none) -> Connector_PinHeader_2.54mm:PinHeader_2x14_P2.54mm_Vertical
- Q1: footprint (none) -> Package_TO_SOT_THT:TO-92_Inline; symbol Transistor_BJT:Q_NPN_BCE -> Transistor_BJT:Q_NPN_CBE
- R1, R2, R3: footprint (none) -> Resistor_THT:R_Axial_DIN0207_L6.3mm_D2.5mm_P10.16mm_Horizontal
Connections:
- net at J4.2 (Pin_2): now also Q1.1 (C); no longer Q1.2 (C)
- net at R2.2, R3.1: now also Q1.2 (B); no longer Q1.1 (B)
Changed lines of the file:
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@@
 			)
 		)
-		(property "Footprint" ""
+		(property "Footprint" "Capacitor_THT:C_Disc_D4.7mm_W2.5mm_P5.00mm"
 			(at 186.3852 107.95 0)
 			(hide yes)
@@
 			)
 		)
-		(property "Footprint" ""
+		(property "Footprint" "Capacitor_THT:C_Disc_D4.7mm_W2.5mm_P5.00mm"
 			(at 135.5852 107.95 0)
 			(hide yes)
@@
 			)
 		)
-		(property "Value" "Conn_01x02_Pin"
+		(property "Value" "LCD Backlight"
 			(at 178.435 66.04 0)
 			(show_name no)
@@
 			)
 		)
-		(property "Footprint" "Package_DIP:DIP-20_W7.62mm"
+		(property "Footprint" "Connector_PinSocket_2.54mm:PinSocket_1x02_P2.54mm_Horizontal"
 			(at 177.8 68.58 0)
 			(hide yes)
@@
 			)
 		)
-		(property "Footprint" "Connector_PinHeader_2.54mm:PinHeader_1x11_P2.54mm_Vertical"
+		(property "Footprint" "Connector_PinSocket_2.54mm:PinSocket_1x11_P2.54mm_Vertical"
 			(at 152.4 38.1 0)
 			(hide yes)
@@
 			)
 		)
-		(property "Footprint" ""
+		(property "Footprint" "Capacitor_THT:C_Disc_D4.7mm_W2.5mm_P5.00mm"
 			(at 125.4252 107.95 0)
 			(hide yes)
@@
 			)
 		)
-		(property "Footprint" ""
+		(property "Footprint" "Capacitor_THT:C_Disc_D4.7mm_W2.5mm_P5.00mm"
 			(at 166.0652 107.95 0)
 			(hide yes)
@@
 			)
 		)
-		(property "Footprint" "Package_DIP:DIP-20_W7.62mm"
+		(property "Footprint" "Connector_FFC-FPC:Hirose_FH12-28S-0.5SH_1x28-1MP_P0.50mm_Horizontal"
 			(at 102.87 82.55 0)
 			(hide yes)
@@
 	)
 	(symbol
-		(lib_id "Transistor_BJT:Q_NPN_BCE")
+		(lib_id "Transistor_BJT:Q_NPN_CBE")
 		(at 189.23 76.2 0)
 		(unit 1)
@@
 			)
 		)
-		(property "Footprint" ""
+		(property "Footprint" "Package_TO_SOT_THT:TO-92_Inline"
 			(at 194.31 73.66 0)
 			(hide yes)
@@
 			)
 		)
-		(property "Description" "NPN transistor, base/collector/emitter"
+		(property "Description" "NPN transistor, collector/base/emitter"
 			(at 189.23 76.2 0)
 			(hide yes)
@@
 			)
 		)
-		(property "Sim.Pins" "1=B 2=C 3=E"
+		(property "Sim.Pins" "1=C 2=B 3=E"
 			(at 189.23 76.2 0)
 			(hide yes)
@@
 	)
 	(symbol
-		(lib_id "Device:C")
+		(lib_id "Device:C_Polarized")
 		(at 151.13 72.39 0)
 		(unit 1)
@@
 		(fields_autoplaced yes)
 		(property "Reference" "C10"
-			(at 154.94 71.1199 0)
+			(at 154.94 70.2309 0)
 			(show_name no)
 			(do_not_autoplace no)
@@
 		)
 		(property "Value" "10uF"
-			(at 154.94 73.6599 0)
+			(at 154.94 72.7709 0)
 			(show_name no)
 			(do_not_autoplace no)
@@
 			)
 		)
-		(property "Footprint" ""
+		(property "Footprint" "Capacitor_THT:CP_Radial_D5.0mm_P2.50mm"
 			(at 152.0952 76.2 0)
 			(hide yes)
@@
 			)
 		)
-		(property "Description" "Unpolarized capacitor"
+		(property "Description" "Polarized capacitor"
 			(at 151.13 72.39 0)
 			(hide yes)
@@
 			)
 		)
-		(property "Footprint" ""
+		(property "Footprint" "Capacitor_THT:C_Disc_D4.7mm_W2.5mm_P5.00mm"
 			(at 196.5452 107.95 0)
 			(hide yes)
@@
 			)
 		)
-		(property "Footprint" "Package_DIP:DIP-20_W7.62mm"
+		(property "Footprint" "Connector_PinHeader_2.54mm:PinHeader_1x02_P2.54mm_Vertical"
 			(at 119.38 40.64 0)
 			(hide yes)
@@
 			)
 		)
-		(property "Footprint" ""
+		(property "Footprint" "Capacitor_THT:C_Disc_D4.7mm_W2.5mm_P5.00mm"
 			(at 155.9052 107.95 0)
 			(hide yes)
@@
 			)
 		)
-		(property "Footprint" ""
+		(property "Footprint" "Resistor_THT:R_Axial_DIN0207_L6.3mm_D2.5mm_P10.16mm_Horizontal"
 			(at 164.592 71.12 90)
 			(hide yes)
@@
 			)
 		)
-		(property "Footprint" ""
+		(property "Footprint" "Capacitor_THT:C_Disc_D4.7mm_W2.5mm_P5.00mm"
 			(at 176.2252 107.95 0)
 			(hide yes)
@@
 			)
 		)
-		(property "Footprint" ""
+		(property "Footprint" "Capacitor_THT:C_Disc_D4.7mm_W2.5mm_P5.00mm"
 			(at 138.1252 76.2 0)
 			(hide yes)
@@
 			)
 		)
-		(property "Footprint" ""
+		(property "Footprint" "Capacitor_THT:C_Disc_D4.7mm_W2.5mm_P5.00mm"
 			(at 145.7452 107.95 0)
 			(hide yes)
@@
 			)
 		)
-		(property "Footprint" ""
+		(property "Footprint" "Resistor_THT:R_Axial_DIN0207_L6.3mm_D2.5mm_P10.16mm_Horizontal"
 			(at 164.592 81.28 90)
 			(hide yes)
@@
 			)
 		)
-		(property "Footprint" ""
+		(property "Footprint" "Connector_PinHeader_2.54mm:PinHeader_2x14_P2.54mm_Vertical"
 			(at 223.52 71.12 0)
 			(hide yes)
@@
 			)
 		)
-		(property "Footprint" ""
+		(property "Footprint" "Resistor_THT:R_Axial_DIN0207_L6.3mm_D2.5mm_P10.16mm_Horizontal"
 			(at 189.992 64.77 90)
 			(hide yes)
@@
 			)
 		)
-		(property "Footprint" "Connector_PinHeader_2.54mm:PinHeader_1x11_P2.54mm_Vertical"
+		(property "Footprint" "Connector_PinSocket_2.54mm:PinSocket_1x11_P2.54mm_Vertical"
 			(at 173.99 38.1 0)
 			(hide yes)
